File: pcb/ird-v17.kicad_pcb (KiCad board)
At the start: 2 copper layers, 25.4 x 30.5 mm, 21 parts, among them J1 AVR-TPI-6, J2 Conn_02x06_Odd_Even, K1 G6K-2, Q1 NPN 10K, U1 ATtiny20-U, U2 TSOP75438WTT, U3 TLVM365R15RDNR

Commit message: Rearrange pins
Parts:
- U2: value TSOP75438WTT -> TSOP75438TT
Connections:
- net OC0A_LED renamed PWMO_LED
- net PA5_RELAY renamed DO_RELAY
- R3 pad 1: TPIDATA -> DO_LED
- U1 pad A3: ADC2_DELAY -> DO_LED
- U1 pad B2: unconnected-(U1-PA6-PadB2) -> DI_SENSE
- U1 pad C1: PA4_SENSE -> AI_DELAY
- U2 pad 3: PA4_SENSE -> DI_SENSE
- VR1 pad 2: ADC2_DELAY -> AI_DELAY
Routing:
- net DO_LED: track 0.00 -> 20.0 mm
- net ADC2_DELAY: track 19.6 -> 0.00 mm, vias 2 -> 0
- net AI_DELAY: track 0.00 -> 17.0 mm, vias 0 -> 2
- net DI_SENSE: track 0.00 -> 16.0 mm, vias 0 -> 2
- net PA4_SENSE: track 15.7 -> 0.00 mm, vias 2 -> 0
- net TPIDATA: track 19.3 -> 7.40 mm
- net GND: track 11.7 -> 13.2 mm

Commit message: PCB update
Parts:
- moved R2 2.79 mm to (36.7, 121.2), turned to 180 degrees
- moved R1 2.03 mm to (38.9, 121.2), turned to 180 degrees
- moved Q1 1.78 mm to (37.0, 124.1)
- moved U2 0.13 mm to (44.5, 126.1), turned to -90 degrees
Connections:
- Q1 pad 2: PWMO_LED -> DO_RELAY
- Q1 pad 3: Net-(D3-A) -> Net-(Q1B-C2)
- Q1 pad 5: DO_RELAY -> PWMO_LED
- Q1 pad 6: Net-(Q1A-C1) -> Net-(D3-A)
- R2 pad 2: Net-(Q1A-C1) -> Net-(Q1B-C2)
Routing:
- net VCC: track 34.9 -> 27.1 mm, vias 9 -> 10
- net Net-(Q1B-C2): track 0.00 -> 4.22 mm
- net Net-(D2-PadC): track 3.66 -> 6.64 mm
- net DI_SENSE: track 16.0 -> 13.4 mm
- net PWMO_LED: track 3.88 -> 5.96 mm
- net Net-(Q1A-C1): track 1.47 -> 0.00 mm
- net Net-(D3-A): track 15.0 -> 15.9 mm
- net AI_DELAY: track 17.0 -> 16.3 mm
- net DO_RELAY: track 7.11 -> 7.83 mm, vias 2 -> 0
- net ~{RESET}: track 14.3 -> 14.8 mm

Commit message: Update to use 5V for consistent ATTINY20 programming
Parts:
- D1: value D_Bridge_-AA+ -> CD-HD2006L
- Q1: value NPN 10K -> MUN5211DW1T1G
- R2: value 27R -> 56R
- R3: value 120R -> 750R
- U1: value ATtiny20-U -> ATtiny20-UUR
- U3: value TLVM365R15RDNR -> TLVM365R1RDNR
